Commit message: added vehicle_interface_node

File: xacro_tutorial/urdf_tutorial/urdf/my_vehicle.xacro (robot description, xacro)
@@ -39,4 +39,9 @@
         <origin rpy="1.5708 0 0"/> <!-- rotate to lay flat -->
       </visual>
+      <inertial>
+        <mass value="1.0"/>
+        <origin xyz="0 0 0" rpy="0 0 0"/>
+        <inertia ixx="0.1" iyy="0.1" izz="0.1" ixy="0.0" ixz="0.0" iyz="0.0"/>
+      </inertial>
     </link>
     <joint name="joint_${name}" type="continuous">
